File: 12vUPS/12vUPS.kicad_sch (KiCad schematic)
At the start: 18 parts, among them J1 INPUT, J2 BATTERY, J3 OUTPUT, J4 ENABLE, J5 START ON BATTERY, K1 VEGHA L08A0212VDC, Q1 BDX53C

Commit message: Update 12vUPS-2025-06-06_224542.zip, 12vUPS-2025-06-06_225111.zip, 12vUPS-2025-06-06_225614.zip, and 28 more files
Parts:
- removed #SW2: SW_Push, symbol Switch:SW_Push
- removed C1: C_Small_US, symbol Device:C_Small_US
- removed C2: 10uF, symbol Device:C_Polarized_Small
- removed J5: START ON BATTERY, Connector_JST:JST_EH_B2B-EH-A_1x02_P2.50mm_Vertical, symbol Connector_Generic:Conn_01x02
- removed R3: 47, Resistor_THT:R_Axial_Power_L48.0mm_W12.5mm_P55.88mm, symbol Device:R
- added D5: D, Diode_THT:D_DO-41_SOD81_P10.16mm_Horizontal, symbol Device:D
- added D6: 4V1, Diode_THT:D_DO-35_SOD27_P7.62mm_Horizontal, symbol Device:D_Zener
- added SW1: BATTERY START, symbol Switch:SW_Push
- D1: value BYW19 -> SF30GG; footprint Package_TO_SOT_THT:TO-220-2_Vertical -> Diode_THT:D_DO-201AD_P15.24mm_Horizontal
- D7: footprint (none) -> IK5PWC:D_IDEAL_with_GND
- J4: footprint Connector_JST:JST_EH_B3B-EH-A_1x03_P2.50mm_Vertical -> Connector_JST:JST_EH_B4B-EH-A_1x04_P2.50mm_Vertical; symbol Connector_Generic:Conn_01x03 -> Connector_Generic:Conn_01x04
- Q1: value BDX53C -> BC337; footprint Package_TO_SOT_THT:TO-220-3_Vertical -> Package_TO_SOT_THT:TO-92_Inline_Wide; symbol Transistor_BJT:Q_NPN_BCE -> Transistor_BJT:BC337
Connections:
- net BATT_IN: now also D7.2 (A), SW1.2; no longer #SW1.1, J4.1 (Pin_1), K1.24
- net ENA: now also J4.3 (Pin_3); no longer J4.2 (Pin_2)
- net GND: no longer #SW1.3 (K), J4.3 (Pin_3)
- net OUT: now also K1.21; no longer D7.1 (K)
- net at RV1.2: now also D6.1 (K); no longer Q1.1 (B)
- net BJT-GND: now reaches D4.2 (A), K1.A2
- net BJT-GND: now also #SW1.3 (K), J4.4 (Pin_4), Q1.1 (C); no longer Q1.2 (C)
- net BATT_START renamed DC-IN-RELE
- net DC-IN-RELE: now also #SW1.1, J4.1 (Pin_1), D5.2 (A), SW1.1; no longer RV1.3
- new net: D6.2 (A), Q1.2 (B)
- new net: D5.1 (K), RV1.3
- new net: D7.1 (K), J4.2 (Pin_2), K1.24
Other:
- moved on the sheet: D1, D7, J1, R1

Commit message: Update 12vUPS-2025-06-08_233608.zip, 12vUPS-2025-06-08_234122.zip, 12vUPS-2025-06-22_122202.zip, and 5 more files
Parts:
- D7: footprint IK5PWC:D_IDEAL_with_GND -> IK5PWC:D_IDEAL_no_GND; symbol IK5PWC:D_Ideal -> IK5PWC:D_Ideal_no_gnd
Connections:
- net GND: no longer D7.3 (GND)
Changed lines of the file:
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@@
-	(wire
-		(pts
-			(xy 105.41 71.12) (xy 105.41 78.74)
-		)
-		(stroke
-			(width 0)
-			(type default)
-		)
-	)
 	(wire
 		(pts
@@
 		(pts
 			(xy 38.1 82.55) (xy 38.1 95.25)
-		)
-		(stroke
-			(width 0)
-			(type default)
-		)
-	)
-	(wire
-		(pts
-			(xy 105.41 78.74) (xy 95.25 78.74)
 		)
 		(stroke
@@
 	)
 	(symbol
-		(lib_id "IK5PWC:D_Ideal")
+		(lib_id "IK5PWC:D_Ideal_no_gnd")
 		(at 105.41 66.04 0)
 		(mirror y)
@@
 			)
 		)
-		(property "Footprint" "IK5PWC:D_IDEAL_with_GND"
+		(property "Footprint" "IK5PWC:D_IDEAL_no_GND"
 			(at 105.41 66.04 0)
 			(effects
@@
 		(pin "2"
 		)
-		(pin "3"
-		)
-		(instances
+		(instances

Commit message: .
Other:
- added sheet Untitled Sheet (monitoring.kicad_sch)
Changed lines of the file:
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@@
+		)
+	)
+	(sheet
+		(at 187.452 137.922)
+		(size 35.56 15.24)
+		(exclude_from_sim no)
+		(in_bom yes)
+		(on_board yes)
+		(dnp no)
+		(fields_autoplaced yes)
+		(stroke
+			(width 0.1524)
+			(type solid)
+		)
+		(fill
+			(color 0 0 0 0.0000)
+		)
+		(property "Sheetname" "Untitled Sheet"
+			(at 187.452 137.2104 0)
+			(effects
+				(font
+					(size 1.27 1.27)
+				)
+				(justify left bottom)
+			)
+		)
+		(property "Sheetfile" "monitoring.kicad_sch"
+			(at 187.452 153.7466 0)
+			(effects
+				(font
+					(size 1.27 1.27)
+				)
+				(justify left top)
+			)
+		)
+		(instances
+			(project "12vUPS"
+				(path "/9d34b600-f815-4c52-bedd-9574651725eb"
+					(page "2")
+				)
+			)
 		)
 	)
