File: 12vUPS/12vUPS.kicad_pcb (KiCad board)
At the start: 2 copper layers, 12 parts, among them J1 INPUT, J2 OUTPUT, J3 BATTERY, K1 VEGHA L08A0212VDC, Q1 BDX53C

Commit message: Update 12vUPS-2025-06-02_174418.zip, 12vUPS-2025-06-06_223532.zip, 12vUPS-2025-06-06_224038.zip, and 9 more files
Parts:
- removed D6: 60CPQ150, Package_TO_SOT_THT:TO-247-3_Vertical
- added D3: LED_Small, LED_THT:LED_D3.0mm, F.Cu at (37.5, 31.5)
- added REF**: MountingHole_3mm, MountingHole:MountingHole_3mm, F.Cu at (82.8, 19.7)
- added REF**: MountingHole_3mm, MountingHole:MountingHole_3mm, F.Cu at (16.1, 73.9)
- added REF**: MountingHole_3mm, MountingHole:MountingHole_3mm, F.Cu at (16.0, 19.6)
- added REF**: MountingHole_3mm, MountingHole:MountingHole_3mm, F.Cu at (82.8, 73.9)
- added RV1: 10K, Potentiometer_THT:Potentiometer_Vishay_T93YA_Vertical, F.Cu at (60.3, 43.5)
- D1: value 30CPF04 -> BYW19; footprint Package_TO_SOT_THT:TO-247-3_Vertical -> Package_TO_SOT_THT:TO-220-2_Vertical
- D2: value LED_Small -> 30CPF04; footprint LED_THT:LED_D3.0mm -> Package_TO_SOT_THT:TO-247-3_Vertical
- D5: value BYW19 -> D_Schottky_Dual_CommonCathode_AKA_Parallel; footprint Package_TO_SOT_THT:TO-220-2_Vertical -> Package_TO_SOT_THT:TO-247-3_Vertical
- J1: footprint TerminalBlock:TerminalBlock_bornier-2_P5.08mm -> TerminalBlock_MetzConnect:TerminalBlock_MetzConnect_Type703_RT10N02HGLU_1x02_P9.52mm_Horizontal
- J2: value OUTPUT -> BATTERY; footprint TerminalBlock:TerminalBlock_bornier-2_P5.08mm -> TerminalBlock_MetzConnect:TerminalBlock_MetzConnect_Type703_RT10N02HGLU_1x02_P9.52mm_Horizontal
- J3: value BATTERY -> OUTPUT; footprint TerminalBlock:TerminalBlock_bornier-2_P5.08mm -> TerminalBlock_MetzConnect:TerminalBlock_MetzConnect_Type703_RT10N02HGLU_1x02_P9.52mm_Horizontal
- K1: footprint Relay_THT:Relay_SPDT_Schrack-RP-II-1-16A-FormC_RM5mm -> IK5PWC:VEGhA L08 12V dc
- R1: value 510 -> 2R7; footprint Resistor_THT:R_Axial_DIN0204_L3.6mm_D1.6mm_P7.62mm_Horizontal -> Resistor_THT:R_Axial_Power_L48.0mm_W12.5mm_P55.88mm
- R2: value 2R7 -> 510; footprint Resistor_THT:R_Axial_Power_L48.0mm_W12.5mm_P55.88mm -> Resistor_THT:R_Axial_DIN0204_L3.6mm_D1.6mm_P7.62mm_Horizontal
- moved D2 117.7 mm to (22.9, 74.3), turned to 90 degrees
- moved R2 114.1 mm to (43.4, 39.2), turned to 90 degrees
- moved D1 110.1 mm to (24.6, 19.2), turned to -90 degrees
- moved J2 99.0 mm to (64.1, 65.0), turned to 0 degrees
- moved K1 92.2 mm to (33.0, 49.3), turned to -90 degrees
- moved R1 88.9 mm to (51.2, 74.9), turned to 90 degrees
- moved D4 88.3 mm to (31.8, 44.3), turned to 0 degrees
- moved J3 88.2 mm to (73.9, 38.0), turned to 90 degrees
- moved Q1 81.1 mm to (33.8, 38.3)
- moved J1 77.1 mm to (21.5, 45.0), turned to -90 degrees
- moved D5 26.1 mm to (73.4, 53.7), turned to 180 degrees
Connections:
- D2 pad 2: Net-(D2-A) -> VCC
- D5 pad 1: Net-(D5-K) -> Net-(D5-A-Pad1)
- D5 pad 2: VCC -> Net-(D5-K)
- J1 pad 1: VCC -> GND
- J1 pad 2: Net-(D4-K) -> VCC
- J2 pad 1: Net-(D1-K) -> Net-(J2-Pin_1)
- J3 pad 1: GND -> Net-(D5-K)
- J3 pad 2: Net-(D4-K) -> GND
- K1 pad 11: Net-(D4-K) -> Net-(D5-K)
- K1 pad 12: Net-(D6-A) -> unconnected-(K1-Pad12)
- K1 pad 14: unconnected-(K1-Pad14)_1 -> Net-(D2-K)
- Q1 pad 2: Net-(D2-K) -> Net-(D3-K)
- R1 pad 1: Net-(R1-Pad1) -> Net-(J2-Pin_1)
- R1 pad 2: Net-(D2-A) -> Net-(D1-K)
- R2 pad 1: Net-(D4-K) -> Net-(R2-Pad1)
- R2 pad 2: Net-(D5-K) -> Net-(D3-A)
Routing:
- net Net-(J2-Pin_1): track 0.00 -> 98.4 mm
- net Net-(D5-K): track 0.00 -> 71.0 mm
- net VCC: track 0.00 -> 57.2 mm
- net Net-(D5-A-Pad1): track 0.00 -> 46.4 mm
- net Net-(D1-K): track 0.00 -> 27.8 mm
- net Net-(R2-Pad1): track 0.00 -> 24.0 mm
- net Net-(D4-A): track 0.00 -> 19.0 mm
- net Net-(D2-K): track 0.00 -> 10.3 mm
- net Net-(D3-K): track 0.00 -> 6.66 mm
- net Net-(D4-K): track 0.00 -> 5.56 mm
- net Net-(D3-A): track 0.00 -> 3.36 mm
- added copper zone on B.Cu, net GND
Other:
- board outline added: 73.2 x 60.8 mm

Commit message: Update #auto_saved_files#, 12vUPS-2025-06-06_223532.zip, 12vUPS-2025-06-07_150941.zip, and 13 more files
Parts:
- added J4: ENABLE, Connector_JST:JST_EH_B3B-EH-A_1x03_P2.50mm_Vertical, F.Cu at (22.4, 40.8)
- D2: footprint Package_TO_SOT_THT:TO-247-3_Vertical -> IK5PWC:30CPF04
- J1, J2, J3: footprint TerminalBlock_MetzConnect:TerminalBlock_MetzConnect_Type703_RT10N02HGLU_1x02_P9.52mm_Horizontal -> IK5PWC:Mammooth_4mm
- moved RV1 40.9 mm to (21.7, 57.3)
- moved R2 23.8 mm to (24.0, 53.0)
- moved D3 21.6 mm to (27.4, 50.6), turned to 90 degrees
- moved J1 20.1 mm to (29.7, 26.7)
- moved D5 17.6 mm to (61.3, 40.8), turned to -90 degrees
- moved J3 13.4 mm to (61.0, 34.5)
- moved Q1 10.3 mm to (41.3, 31.1), turned to -90 degrees
- moved D1 8.37 mm to (33.0, 19.2), turned to 180 degrees
- moved REF** 8.02 mm to (74.8, 19.8)
- moved REF** 8.00 mm to (74.8, 73.9)
- moved J2 3.38 mm to (61.0, 66.3), turned to 90 degrees
- moved D2 1.48 mm to (24.4, 74.1)
- moved R1 0.14 mm to (51.2, 74.7)
Connections:
- net Net-(D4-A) renamed /A2
- net Net-(D4-K) renamed /A1
- net Net-(J2-Pin_1) renamed /+12V
Routing:
- net /+12V: track 98.4 -> 69.0 mm
- net Net-(D3-K): track 6.66 -> 29.0 mm
- net VCC: track 57.2 -> 78.2 mm
- net Net-(R2-Pad1): track 24.0 -> 4.43 mm
- net Net-(D5-K): track 71.0 -> 57.1 mm
- net Net-(D1-K): track 27.8 -> 19.1 mm
- net /A1: track 5.56 -> 14.0 mm
- net Net-(D2-K): track 10.3 -> 13.0 mm
- net /A2: track 19.0 -> 21.5 mm
- net Net-(D3-A): track 3.36 -> 5.43 mm
Other:
- board size 73.2 x 60.8 mm -> 65.4 x 60.8 mm
- board text added: "2025"
- board text added: "IK5PWC"
