File: 12vUPS/_autosave-12vUPS.kicad_sch (KiCad schematic)
At the start: 15 parts, among them J1 INPUT, J2 BATTERY, J3 OUTPUT, J4 ENABLE, K1 VEGHA L08A0212VDC, Q1 BDX53C

Commit message: Update #auto_saved_files#, 12vUPS-2025-06-06_223532.zip, 12vUPS-2025-06-07_150941.zip, and 13 more files
Connections:
- net A2: now reaches D4.2 (A), K1.A2, Q1.1 (C)
- net ENA renamed A1
Changed lines of the file:
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@@
+		)
+	)
+	(label "A2"
+		(at 144.78 88.9 0)
+		(effects
+			(font
+				(size 1.27 1.27)
+			)
+			(justify left bottom)
 		)
 	)
@@
 		(effects
 			(font
+				(size 1.27 1.27)
+			)
+			(justify right bottom)
+		)
+	)
+	(label "A1"
+		(at 128.27 88.9 180)
+		(effects
+			(font
