File: 12vUPS/_autosave-12vUPS.kicad_sch (KiCad schematic)
At the start: 18 parts, among them J1 INPUT, J2 BATTERY, J3 OUTPUT, J4 ENABLE, J5 START ON BATTERY, K1 VEGHA L08A0212VDC, Q1 BDX53C

Commit message: Update #auto_saved_files#, 12vUPS-2025-06-02_175555.zip, 12vUPS-2025-06-02_180136.zip, and 18 more files
Parts:
- removed #SW2: SW_Push, symbol Switch:SW_Push
- removed C1: C_Small_US, symbol Device:C_Small_US
- removed C2: 10uF, symbol Device:C_Polarized_Small
- removed J5: START ON BATTERY, Connector_JST:JST_EH_B2B-EH-A_1x02_P2.50mm_Vertical, symbol Connector_Generic:Conn_01x02
- removed R3: 47, Resistor_THT:R_Axial_Power_L48.0mm_W12.5mm_P55.88mm, symbol Device:R
- added R2: 510, Resistor_THT:R_Axial_DIN0204_L3.6mm_D1.6mm_P7.62mm_Horizontal, symbol Device:R
- D1: value BYW19 -> SF30GG; footprint Package_TO_SOT_THT:TO-220-2_Vertical -> Diode_THT:D_DO-201AD_P15.24mm_Horizontal
- D7: footprint (none) -> IK5PWC:D_IDEAL_with_GND
Connections:
- net BATT_IN: now also D7.2 (A); no longer #SW1.1, J4.1 (Pin_1), K1.24
- net GND: no longer #SW1.3 (K), J4.3 (Pin_3)
- net OUT: now also K1.21; no longer D7.1 (K)
- net at Q1.1 (B): now also R2.1; no longer RV1.2
- net BJT-GND: now reaches D4.2 (A), K1.A2, Q1.2 (C)
- net BJT-GND: now also #SW1.3 (K), J4.3 (Pin_3)
- net BATT_START renamed DC-IN-RELE
- net DC-IN-RELE: now also #SW1.1, D7.1 (K), J4.1 (Pin_1), K1.24
- new net: R2.2, RV1.2
Other:
- moved on the sheet: D1, D7, J1, R1, RV1

Commit message: Update 12vUPS-2025-06-06_224542.zip, 12vUPS-2025-06-06_225111.zip, 12vUPS-2025-06-06_225614.zip, and 28 more files
Parts:
- removed R2: 510, Resistor_THT:R_Axial_DIN0204_L3.6mm_D1.6mm_P7.62mm_Horizontal, symbol Device:R
- added D5: D, Diode_THT:D_DO-41_SOD81_P10.16mm_Horizontal, symbol Device:D
- added D6: 4V1, Diode_THT:D_DO-35_SOD27_P7.62mm_Horizontal, symbol Device:D_Zener
- added SW1: BATTERY START, symbol Switch:SW_Push
- J4: footprint Connector_JST:JST_EH_B3B-EH-A_1x03_P2.50mm_Vertical -> Connector_JST:JST_EH_B4B-EH-A_1x04_P2.50mm_Vertical; symbol Connector_Generic:Conn_01x03 -> Connector_Generic:Conn_01x04
- Q1: value BDX53C -> BC337; footprint Package_TO_SOT_THT:TO-220-3_Vertical -> Package_TO_SOT_THT:TO-92_Inline_Wide; symbol Transistor_BJT:Q_NPN_BCE -> Transistor_BJT:BC337
Connections:
- net BATT_IN: now also SW1.2
- net BJT-GND: now also J4.4 (Pin_4), Q1.1 (C); no longer J4.3 (Pin_3), Q1.2 (C)
- net DC-IN-RELE: now also D5.2 (A), SW1.1; no longer D7.1 (K), K1.24, RV1.3
- net ENA: now also J4.3 (Pin_3); no longer J4.2 (Pin_2)
- net at RV1.2: now also D6.1 (K)
- new net: D6.2 (A), Q1.2 (B)
- new net: D5.1 (K), RV1.3
- new net: D7.1 (K), J4.2 (Pin_2), K1.24
Other:
- moved on the sheet: RV1
