File: 12vUPS-modules/12vUPS-modules.kicad_sch (KiCad schematic)
At the start: 16 parts, among them J1 INPUT, J2 BATTERY, J3 OUTPUT, J4 ENABLE, K1 VEGHA L08A0212VDC, Q1 BC337, SW1 BATTERY START

Commit message: Update 12vUPS-modles.kicad_prl, 12vUPS-modules-2025-07-13_234921.zip, 12vUPS-modules-2025-07-14_221001.zip, and 54 more files
Other:
- removed sheet Untitled Sheet
Changed lines of the file:
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@@
-		)
-	)
-	(sheet
-		(at 187.452 137.922)
-		(size 35.56 15.24)
-		(exclude_from_sim no)
-		(in_bom yes)
-		(on_board yes)
-		(dnp no)
-		(fields_autoplaced yes)
-		(stroke
-			(width 0.1524)
-			(type solid)
-		)
-		(fill
-			(color 0 0 0 0.0000)
-		)
-		(property "Sheetname" "Untitled Sheet"
-			(at 187.452 137.2104 0)
-			(effects
-				(font
-					(size 1.27 1.27)
-				)
-				(justify left bottom)
-			)
-		)
-		(property "Sheetfile" "monitoring.kicad_sch"
-			(at 187.452 153.7466 0)
-			(effects
-				(font
-					(size 1.27 1.27)
-				)
-				(justify left top)
-			)
-		)
-		(instances
-			(project "12vUPS"
-				(path "/9d34b600-f815-4c52-bedd-9574651725eb"
-					(page "2")
-				)
-			)
 		)
 	)
