File: Kicad/monitoring/monitoring.kicad_sch (KiCad schematic)
At the start: 20 parts, among them J1 Conn_01x04, J2 Conn_01x04, J3 Conn_01x04, J4 Conn_01x03, J5 Conn_01x05, J6 Conn_01x05, J7 Screw_Terminal_01x03, U1 4052, U3 L7805, U4 L7805

Commit message: Update 12vUPS-modles.kicad_prl, 12vUPS-modules-2025-07-13_234921.zip, 12vUPS-modules-2025-07-14_221001.zip, and 69 more files
Parts:
- J1: value Conn_01x04 -> Module1
- J2: value Conn_01x04 -> Module2
- J3: value Conn_01x04 -> Module3
- J4: value Conn_01x03 -> buttons
- J5, J6: value Conn_01x05 -> Display
- J7: value Screw_Terminal_01x03 -> DC_in_outout
Connections:
- net +5VA: no longer R3.2, R7.2
- net LCD_D4: now also J5.5 (Pin_5); no longer J5.1 (Pin_1)
- net LCD_D5: now also J5.4 (Pin_4); no longer J5.2 (Pin_2)
- net LCD_D7: now also J5.2 (Pin_2); no longer J5.4 (Pin_4)
- net VCC: now also R3.2
- net at A1.5 (+5V): now also R7.2
- net at R2.2: now also J5.1 (Pin_1); no longer J5.5 (Pin_5)
- net dc_out renamed ps_out
- no-connect marks 11 -> 10
Other:
- moved on the sheet: J5, R3, R4

Commit message: Update #auto_saved_files#, Arduino_UNO_R2.kicad_mod, fp-info-cache, and 9 more files
Parts:
- A1: footprint Module:Arduino_UNO_R2 -> custom_lib:Arduino_UNO_R2
Connections:
- net +5VA: now also R7.2
- net at A1.5 (+5V): no longer R7.2
- no-connect marks 10 -> 11
Changed lines of the file:
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@@
+	)
+	(junction
+		(at 177.8 54.61)
+		(diameter 0)
+		(color 0 0 0 0)
 	)
 	(junction
@@
 	)
 	(no_connect
+		(at 135.89 44.45)
+	)
+	(no_connect
 		(at 118.11 54.61)
 	)
@@
 	(wire
 		(pts
+			(xy 154.94 54.61) (xy 154.94 55.88)
+		)
+		(stroke
+			(width 0)
+			(type default)
+		)
+	)
+	(wire
+		(pts
 			(xy 73.66 90.17) (xy 82.55 90.17)
 		)
@@
 	(wire
 		(pts
+			(xy 177.8 54.61) (xy 154.94 54.61)
+		)
+		(stroke
+			(width 0)
+			(type default)
+		)
+	)
+	(wire
+		(pts
 			(xy 229.87 107.95) (xy 232.41 107.95)
 		)
@@
 	(wire
 		(pts
-			(xy 154.94 44.45) (xy 154.94 55.88)
-		)
-		(stroke
-			(width 0)
-			(type default)
-		)
-	)
-	(wire
-		(pts
 			(xy 190.5 69.85) (xy 214.63 69.85)
-		)
-		(stroke
-			(width 0)
-			(type default)
-		)
-	)
-	(wire
-		(pts
-			(xy 135.89 44.45) (xy 154.94 44.45)
 		)
 		(stroke
@@
 			)
 		)
-		(property "Footprint" "Module:Arduino_UNO_R2"
+		(property "Footprint" "custom_lib:Arduino_UNO_R2"
 			(at 130.81 69.85 0)
 			(effects

Commit message: Ready for 1st test
Connections:
- net BCD-1: now also U1.9 (B); no longer U1.10 (A)
- net BCD-2: now also U1.10 (A); no longer U1.9 (B)
Changed lines of the file:
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@@
-	(wire
-		(pts
-			(xy 198.12 90.17) (xy 198.12 109.22)
-		)
-		(stroke
-			(width 0)
-			(type default)
-		)
-	)
 	(wire
 		(pts
@@
 	(wire
 		(pts
+			(xy 194.31 92.71) (xy 194.31 109.22)
+		)
+		(stroke
+			(width 0)
+			(type default)
+		)
+	)
+	(wire
+		(pts
 			(xy 60.96 180.34) (xy 60.96 181.61)
 		)
@@
 	(wire
 		(pts
-			(xy 190.5 92.71) (xy 196.85 92.71)
+			(xy 190.5 92.71) (xy 194.31 92.71)
 		)
 		(stroke
@@
 	(wire
 		(pts
+			(xy 198.12 90.17) (xy 198.12 106.68)
+		)
+		(stroke
+			(width 0)
+			(type default)
+		)
+	)
+	(wire
+		(pts
 			(xy 163.83 102.87) (xy 219.71 102.87)
 		)
@@
 	(wire
 		(pts
-			(xy 196.85 92.71) (xy 196.85 106.68)
-		)
-		(stroke
-			(width 0)
-			(type default)
-		)
-	)
-	(wire
-		(pts
 			(xy 220.98 95.25) (xy 226.06 95.25)
 		)
@@
 	(wire
 		(pts
-			(xy 107.95 109.22) (xy 198.12 109.22)
+			(xy 107.95 109.22) (xy 194.31 109.22)
 		)
 		(stroke
@@
 	(wire
 		(pts
-			(xy 110.49 106.68) (xy 196.85 106.68)
+			(xy 110.49 106.68) (xy 198.12 106.68)
 		)
 		(stroke
@@
 	)
 	(label "BCD-1"
+		(at 190.5 92.71 0)
+		(effects
+			(font
+				(size 1.27 1.27)
+			)
+			(justify left bottom)
+		)
+	)
+	(label "BCD-2"
 		(at 190.5 90.17 0)
 		(effects
 			(font
-				(size 1.27 1.27)
-			)
-			(justify left bottom)
-		)
-	)
-	(label "BCD-2"
-		(at 190.5 92.71 0)
-		(effects
-			(font
