File: Kicad/monitoring/monitoring.kicad_pcb (KiCad board)
At the start: 2 copper layers, 98.7 x 51.1 mm, 19 parts, among them J1 Module1, J2 Module2, J3 Module3, J4 buttons, J5 Display, J6 Display, J7 DC_in_outout, U1 4052, U3 L7805, U4 L7805

Commit message: Update #auto_saved_files#, Arduino_UNO_R2.kicad_mod, fp-info-cache, and 9 more files
Parts:
- A1: footprint Module:Arduino_UNO_R2 -> custom_lib:Arduino_UNO_R2
- moved R7 9.23 mm to (75.0, 66.3), turned to 90 degrees
- moved R6 6.36 mm to (72.2, 58.5)
- moved U3 4.42 mm to (123.3, 59.3), turned to -90 degrees
Connections:
- A1 pad 5: Net-(A1-+5V) -> unconnected-(A1-+5V-Pad5)
- R7 pad 2: Net-(A1-+5V) -> +5VA
Routing:
- net +5VA: track 144.5 -> 200.6 mm
- net /COMMON: track 36.1 -> 12.6 mm
- net Net-(A1-+5V): track 10.1 -> 0.00 mm
- net /UP: track 15.4 -> 7.26 mm
- net VCC: track 105.8 -> 111.4 mm, vias 2 -> 0
- net /ps_out: track 34.5 -> 31.3 mm

Commit message: Ready for 1st test
Parts:
- moved J7 114.7 mm to (40.2, 116.5), turned to 180 degrees
- moved U4 109.4 mm to (48.5, 116.8), turned to 0 degrees
- moved R2 99.7 mm to (49.5, 109.6), turned to 180 degrees
- moved RV2 97.3 mm to (66.6, 114.2), turned to 0 degrees
- moved J5 96.9 mm to (45.5, 105.0), turned to 180 degrees
- moved R1 90.7 mm to (35.4, 90.8), turned to 0 degrees
- moved R5 86.2 mm to (35.4, 86.1), turned to 0 degrees
- moved J6 83.7 mm to (69.2, 105.0), turned to 180 degrees
- moved R3 82.1 mm to (35.4, 81.4), turned to 0 degrees
- moved U1 78.7 mm to (32.9, 72.6), turned to 90 degrees
- moved R4 78.4 mm to (35.4, 76.6), turned to 0 degrees
- moved J3 78.1 mm to (29.7, 30.7), turned to 0 degrees
- moved U3 58.6 mm to (73.5, 90.1), turned to 90 degrees
- moved J2 55.1 mm to (47.1, 30.7), turned to 0 degrees
- moved J4 36.3 mm to (63.5, 29.8), turned to 0 degrees
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Routing:
- net +5VA: track 200.6 -> 165.4 mm
- net /COMMON: track 12.6 -> 46.7 mm, vias 0 -> 2
- net /m1_Iout: track 22.4 -> 27.8 mm
- net VCC: track 111.4 -> 106.3 mm
- net /BCD-2: track 34.7 -> 38.7 mm
- net /BCD-1: track 34.7 -> 37.8 mm
- net /m1_Ibat: track 28.8 -> 31.9 mm
- net /m3_Ibat: track 61.4 -> 59.5 mm
- net /ps_out: track 31.3 -> 33.2 mm
- net /m2_Ibat: track 68.3 -> 66.9 mm, vias 4 -> 2
- net /m3_Vbat: track 18.9 -> 17.8 mm, vias 0 -> 2
- net Net-(A1-A1): track 41.0 -> 42.0 mm
- net /LCD_D7: track 11.0 -> 11.9 mm
- net /m2_Vbat: track 26.3 -> 25.5 mm
- net /m2_Iout: track 65.1 -> 64.4 mm, vias 2 -> 0
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Other:
- board size 98.7 x 51.1 mm -> 51.1 x 98.7 mm
- board text added: "IK5PWC 2025"

Commit message: Update .cproject, .project, UPSMonitor.ino, and 29 more files
Parts:
- removed R6: 10K, Resistor_THT:R_Axial_DIN0204_L3.6mm_D1.6mm_P7.62mm_Horizontal
- added C1: 100 nF, Capacitor_THT:C_Disc_D4.7mm_W2.5mm_P5.00mm, F.Cu at (44.5, 103.3)
- added C3: 220 uF, Capacitor_THT:CP_Radial_D10.0mm_P5.00mm, F.Cu at (61.6, 79.1)
- added C4: 100 nF, Capacitor_THT:C_Disc_D4.7mm_W2.5mm_P5.00mm, F.Cu at (63.4, 37.9)
- J4: footprint Connector_JST:JST_XH_B3B-XH-A_1x03_P2.50mm_Vertical -> Connector_JST:JST_XH_B2B-XH-A_1x02_P2.50mm_Vertical
- moved U3 20.6 mm to (66.3, 70.8)
- moved R2 11.5 mm to (39.9, 103.3)
- moved R3 11.1 mm to (27.8, 73.3)
- moved A1 11.1 mm to (63.0, 39.7)
- moved J2 11.1 mm to (39.5, 22.7)
- moved J7 11.1 mm to (32.5, 108.5)
- moved RV2 11.1 mm to (59.0, 106.2)
- moved U1 11.1 mm to (25.2, 64.5)
- moved U4 11.1 mm to (40.9, 108.7)
- moved J3 11.1 mm to (22.0, 22.7)
- moved R1 11.1 mm to (27.8, 82.8)
- moved R4 11.1 mm to (27.8, 68.6)
- moved R5 11.1 mm to (27.8, 78.0)
- moved J5 11.1 mm to (37.8, 96.9)
- moved J6 11.1 mm to (61.6, 96.9)
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Connections:
- net /COMMON renamed /PUSH
- net /dc_Vin renamed /ps_Vin
- J1 pad 1: +5VA -> /m1_Vbat
- J1 pad 2: /m1_Iout -> +5VA
- J1 pad 3: /m1_Ibat -> /m1_Iout
- J1 pad 4: /m1_Vbat -> /m1_Ibat
- J2 pad 1: +5VA -> /m2_Vbat
- J2 pad 2: /m2_Iout -> +5VA
- J2 pad 3: /m2_Ibat -> /m2_Iout
- J2 pad 4: /m2_Vbat -> /m2_Ibat
- J3 pad 1: +5VA -> /m3_Vbat
- J3 pad 2: /m3_Iout -> +5VA
- J3 pad 3: /m3_Ibat -> /m3_Iout
- J3 pad 4: /m3_Vbat -> /m3_Ibat
- J4 pad 1: /UP -> GND
Routing:
- net /m1_Vbat: track 24.2 -> 43.1 mm
- net VCC: track 106.3 -> 125.2 mm
- net +5VA: track 165.4 -> 154.0 mm
- net /UP: track 7.26 -> 0.00 mm
- net /m1_Ibat: track 31.9 -> 27.1 mm
- net /m2_Vbat: track 25.5 -> 22.0 mm, vias 0 -> 2
- net Net-(A1-A0): track 24.0 -> 20.8 mm
- net /m1_Iout: track 27.8 -> 24.8 mm
- net /m3_Vbat: track 17.8 -> 20.8 mm
- net +5VD: track 33.0 -> 35.7 mm
- net /LCD_EN: track 11.7 -> 14.3 mm
- net /m2_Iout: track 64.4 -> 61.9 mm
- net Net-(A1-A1): track 42.0 -> 39.6 mm
- net /m2_Ibat: track 66.9 -> 64.6 mm
- net /PUSH: track 46.7 -> 45.1 mm, vias 2 -> 0
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
Commit message: Update UPSMonitor.ino, datatypes.h, io.cpp, and 18 more files
Parts:
- removed R7: 10K, Resistor_THT:R_Axial_DIN0204_L3.6mm_D1.6mm_P7.62mm_Horizontal
- added RN1: 4K7, Resistor_THT:R_Array_SIP10, F.Cu at (47.9, 80.0)
- R1, R3: value 3K3 -> 3K
- moved J3 93.3 mm to (79.2, 96.4)
- moved J7 89.8 mm to (121.7, 97.7), turned to -90 degrees
- moved U4 83.3 mm to (121.9, 89.3), turned to 90 degrees
- moved J4 81.3 mm to (64.2, 104.9)
- moved R2 77.7 mm to (116.5, 90.3), turned to -90 degrees
- moved C1 74.0 mm to (116.4, 85.7), turned to 90 degrees
- moved J5 72.4 mm to (110.1, 92.4), turned to -90 degrees
- moved R3 70.2 mm to (97.2, 83.5), turned to 90 degrees
- moved RV2 69.7 mm to (119.3, 71.2), turned to 90 degrees
- moved R4 68.0 mm to (94.2, 83.4), turned to 90 degrees
- moved C4 67.4 mm to (70.1, 105.0), turned to 0 degrees
- moved R1 63.7 mm to (91.2, 76.9), turned to -90 degrees
- moved R5 60.8 mm to (88.6, 76.9), turned to -90 degrees
- moved J2 57.8 mm to (70.2, 71.6)
- moved J6 56.1 mm to (110.1, 68.6), turned to -90 degrees
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Connections:
- net /dc_Vout renamed /ups_Vout
- net /ps_out renamed Net-(J7-Pin_2)
- J4 pad 1: GND -> +5VA
- R1 pad 1: /ps_Vin -> /ps_Vout
- R5 pad 1: /ps_Vin -> /ps_Vout
- U1 pad 1: /m3_Iout -> /m1_Ibat
- U1 pad 11: /m2_Ibat -> /ps_Vout
- U1 pad 12: /m1_Iout -> /m2_Ibat
- U1 pad 14: /m1_Ibat -> /m2_Iout
- U1 pad 15: /m2_Iout -> /m1_Iout
- U1 pad 2: /ps_Vin -> /m3_Iout
Routing:
- net /m2_Ibat: track 64.6 -> 6.84 mm, vias 2 -> 0
- net /m2_Iout: track 61.9 -> 8.00 mm
- net /m3_Ibat: track 58.8 -> 16.7 mm
- net /PUSH: track 45.1 -> 14.7 mm
- net /m3_Iout: track 50.2 -> 21.3 mm
- net /m1_Vbat: track 43.1 -> 17.2 mm, vias 2 -> 0
- net /m2_Vbat: track 22.0 -> 44.9 mm
- net /BCD-2: track 38.7 -> 16.3 mm
- net /ps_Vin: track 20.2 -> 0.00 mm
- net Net-(J7-Pin_2): track 33.2 -> 51.1 mm
- net /BCD-1: track 37.8 -> 20.6 mm
- net +5VA: track 154.0 -> 137.9 mm, vias 0 -> 2
- net /m1_Ibat: track 27.1 -> 12.3 mm
- net /ps_Vout: track 0.00 -> 13.1 mm
- net /m3_Vbat: track 20.8 -> 33.7 mm, vias 2 -> 0
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Other:
- board size 51.1 x 98.7 mm -> 84.5 x 51.1 mm
- board text added: "2025"
- board text added: "IK5PWC"
- board text removed: "IK5PWC 2025"

Commit message: Update .sproject, io.cpp, io.h, and 29 more files
Parts:
- added R6: 100K, Resistor_THT:R_Axial_DIN0204_L3.6mm_D1.6mm_P7.62mm_Horizontal, F.Cu at (54.8, 62.9)
- added R7: 100K, Resistor_THT:R_Axial_DIN0204_L3.6mm_D1.6mm_P7.62mm_Horizontal, F.Cu at (54.8, 65.5)
- moved J7 89.1 mm to (32.6, 101.8), turned to 180 degrees
- moved U4 81.9 mm to (41.0, 102.1), turned to 0 degrees
- moved R2 76.8 mm to (40.0, 96.7), turned to 180 degrees
- moved C1 72.7 mm to (44.6, 96.6), turned to 0 degrees
- moved J5 72.2 mm to (37.9, 90.3), turned to 180 degrees
- moved J4 71.9 mm to (25.4, 44.4), turned to 90 degrees
- moved C4 70.7 mm to (25.3, 50.3), turned to -90 degrees
- moved RV2 66.6 mm to (59.1, 99.5), turned to 0 degrees
- moved J1 60.0 mm to (33.9, 44.8), turned to -90 degrees
- moved J3 58.5 mm to (33.9, 59.4), turned to -90 degrees
- moved J6 53.0 mm to (61.7, 90.3), turned to 180 degrees
- moved RN1 52.0 mm to (50.3, 28.1), turned to 180 degrees
- moved R3 50.7 mm to (46.8, 77.4), turned to 0 degrees
- moved R4 48.1 mm to (46.9, 74.3), turned to 0 degrees
- moved U1 44.8 mm to (44.3, 47.7), turned to 0 degrees
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Routing:
- net /ps_Vout: track 13.1 -> 17.4 mm
- net /BCD-1: track 20.6 -> 23.5 mm
- net /BCD-2: track 16.3 -> 19.2 mm
- net /m2_Vbat: track 44.9 -> 42.1 mm
- net +5VA: track 137.9 -> 135.5 mm
- net /m2_Ibat: track 6.84 -> 8.84 mm
- net /LCD_RS: track 14.3 -> 16.2 mm
- net /m2_Iout: track 8.00 -> 7.29 mm
Other:
- board size 84.5 x 51.1 mm -> 51.1 x 84.5 mm

Commit message: Update .sproject, params.h, SensorBoard-2025-07-29_231028.zip, and 10 more files
Routing:
- net /m2_Vbat: track 42.1 -> 42.6 mm
Changed lines of the file:
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@@
 	)
 	(segment
-		(start 51.5195 36.776)
-		(end 51.5715 36.828)
+		(start 32.625 37.375)
+		(end 51.674 37.375)
 		(width 0.2)
 		(layer "F.Cu")
@@
 	)
 	(segment
-		(start 32.6515 37.376)
-		(end 32.6315 37.396)
+		(start 51.674 37.375)
+		(end 51.675 37.376)
 		(width 0.2)
 		(layer "F.Cu")
 		(net 7)
 	)
-	(segment
-		(start 51.5115 37.376)
-		(end 32.6515 37.376)
-		(width 0.2)
-		(layer "F.Cu")
-		(net 7)
-	)
 	(via
-		(at 51.5115 37.376)
+		(at 51.675 37.376)
 		(size 2)
 		(drill 0.8)
@@
 	)
 	(via
-		(at 32.6315 37.396)
+		(at 32.625 37.375)
 		(size 2)
 		(drill 0.8)
 		(layers "F.Cu" "B.Cu")
+		(teardrops
+			(best_length_ratio 0.5)
+			(max_length 1)
+			(best_width_ratio 1)
+			(max_width 2)
+			(curved_edges no)
+			(filter_ratio 1)
+			(enabled no)
+			(allow_two_segments yes)
+			(prefer_zone_connections yes)
+		)
+		(net 7)
+	)
+	(segment
+		(start 32.625 37.375)
+		(end 32.5855 37.3355)
+		(width 0.75)
+		(layer "B.Cu")
+		(net 7)
+	)
+	(segment
+		(start 32.5855 33.0255)
+		(end 32.5855 36.76)
+		(width 0.75)
+		(layer "B.Cu")
 		(net 7)
 	)
@@
 	)
 	(segment
-		(start 51.5115 37.376)
-		(end 53.6015 37.376)
-		(width 0.75)
-		(layer "B.Cu")
-		(net 7)
-	)
-	(segment
-		(start 32.5855 33.0255)
-		(end 32.5855 36.76)
-		(width 0.75)
-		(layer "B.Cu")
-		(net 7)
-	)
-	(segment
-		(start 32.6015 36.776)
-		(end 32.6215 36.796)
-		(width 0.75)
-		(layer "B.Cu")
-		(net 7)
-	)
-	(segment
 		(start 32.4915 28.111)
 		(end 32.4915 32.9315)
@@
 	)
 	(segment
+		(start 32.5855 37.3355)
+		(end 32.5855 36.76)
+		(width 0.75)
+		(layer "B.Cu")
+		(net 7)
+	)
+	(segment
+		(start 32.4915 32.9315)
+		(end 32.5855 33.0255)
+		(width 0.75)
+		(layer "B.Cu")
+		(net 7)
+	)
+	(segment
 		(start 53.6015 37.376)
 		(end 58.95 42.7245)
@@
 	)
 	(segment
-		(start 51.5795 36.836)
-		(end 51.5715 36.828)
-		(width 0.75)
-		(layer "B.Cu")
-		(net 7)
-	)
-	(segment
-		(start 32.4915 32.9315)
-		(end 32.5855 33.0255)
-		(width 0.75)
-		(layer "B.Cu")
-		(net 7)
-	)
-	(segment
 		(start 32.5855 36.76)
 		(end 32.6015 36.776)
+		(width 0.75)
+		(layer "B.Cu")
+		(net 7)
+	)
+	(segment
+		(start 51.675 37.376)
+		(end 53.6015 37.376)
 		(width 0.75)
 		(layer "B.Cu")
@@
 		(hatch edge 0.5)
 		(connect_pads thru_hole_only
-			(clearance 0.5)
+			(clearance 0.7)
 		)
 		(min_thickness 0.25)
@@
 		(polygon
 			(pts
-				(xy 45.675 86.325) (xy 43.25 86.325) (xy 43.25 85.55) (xy 43.725 85.075) (xy 43.725 85.025) (xy 44.375 85.025)
+				(xy 52.94 88.64) (xy 50.515 88.64) (xy 50.515 87.865) (xy 50.99 87.39) (xy 50.99 87.34) (xy 51.64 87.34)
 			)
 		)

Commit message: Update fp-info-cache, monitoring-2025-07-18_201733.zip, monitoring-2025-07-18_212227.zip, and 5 more files
Parts:
- RN1: footprint Resistor_THT:R_Array_SIP10 -> Resistor_THT:R_Array_SIP8
- moved RN1 5.04 mm to (45.2, 28.1)
Connections:
- RN1 pad 3: unconnected-(RN1-R2-Pad3) -> Net-(A1-A0)
- RN1 pad 4: unconnected-(RN1-R3-Pad4) -> Net-(A1-A1)
- RN1 pad 5: Net-(A1-A0) -> /m1_Vbat
- RN1 pad 6: Net-(A1-A1) -> /m2_Vbat
- RN1 pad 7: /m1_Vbat -> /m3_Vbat
- RN1 pad 8: /m2_Vbat -> /PUSH
Changed lines of the file:
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@@
 	(net 34 "/ups_Vout")
 	(net 35 "unconnected-(RN1-R1-Pad2)")
-	(net 36 "unconnected-(RN1-R2-Pad3)")
-	(net 37 "unconnected-(RN1-R3-Pad4)")
 	(footprint "Potentiometer_THT:Potentiometer_Bourns_3296W_Vertical"
 		(layer "F.Cu")
@@
 		)
 	)
-	(footprint "Resistor_THT:R_Array_SIP10"
+	(footprint "Resistor_THT:R_Array_SIP8"
 		(layer "F.Cu")
-		(at 50.2715 28.111 180)
-		(descr "10-pin Resistor SIP pack")
+		(at 45.23 28.08 180)
+		(descr "8-pin Resistor SIP pack")
 		(tags "R")
 		(property "Reference" "RN1"
-			(at 12.7 -2.31 0)
+			(at 10.16 -2.31 180)
 			(layer "F.SilkS")
 			(effects
@@
 		)
 		(property "Value" "4K7"
-			(at 12.7 2.31 0)
+			(at 10.16 2.31 180)
 			(layer "F.Fab")
 			(effects
@@
 		)
 		(property "Datasheet" "http://www.vishay.com/docs/31509/csc.pdf"
-			(at 0 0 0)
+			(at 0 0 180)
 			(layer "F.Fab")
 			(hide yes)
@@
 			)
 		)
-		(property "Description" "9 resistor network, star topology, bussed resistors, small symbol"
-			(at 0 0 0)
+		(property "Description" "7 resistor network, star topology, bussed resistors, small symbol"
+			(at 0 0 180)
 			(layer "F.Fab")
 			(hide yes)
@@
 		(attr through_hole)
 		(fp_line
-			(start 24.21 1.31)
-			(end 24.21 -1.31)
+			(start 19.13 1.31)
+			(end 19.13 -1.31)
 			(stroke
 				(width 0.12)
@@
 		)
 		(fp_line
-			(start 24.21 -1.31)
+			(start 19.13 -1.31)
 			(end -1.35 -1.31)
 			(stroke
@@
 		(fp_line
 			(start -1.35 1.31)
-			(end 24.21 1.31)
+			(end 19.13 1.31)
 			(stroke
 				(width 0.12)
@@
 		)
 		(fp_line
-			(start 24.46 1.56)
-			(end 24.46 -1.56)
+			(start 19.38 1.56)
+			(end 19.38 -1.56)
 			(stroke
 				(width 0.05)
@@
 		)
 		(fp_line
-			(start 24.46 -1.56)
+			(start 19.38 -1.56)
 			(end -1.6 -1.56)
 			(stroke
@@
 		(fp_line
 			(start -1.6 1.56)
-			(end 24.46 1.56)
+			(end 19.38 1.56)
 			(stroke
 				(width 0.05)
@@
 		)
 		(fp_line
-			(start 24.15 1.25)
-			(end 24.15 -1.25)
+			(start 19.07 1.25)
+			(end 19.07 -1.25)
 			(stroke
 				(width 0.1)
@@
 		)
 		(fp_line
-			(start 24.15 -1.25)
+			(start 19.07 -1.25)
 			(end -1.29 -1.25)
 			(stroke
@@
 		(fp_line
 			(start -1.29 1.25)
-			(end 24.15 1.25)
+			(end 19.07 1.25)
 			(stroke
 				(width 0.1)
@@
 		)
 		(fp_text user "${REFERENCE}"
-			(at 12.7 0 0)
+			(at 10.16 0 180)
 			(layer "F.Fab")
 			(effects
@@
 			(layers "*.Cu" "*.Mask")
 			(remove_unused_layers no)
-			(net 36 "unconnected-(RN1-R2-Pad3)")
+			(net 18 "Net-(A1-A0)")
 			(pinfunction "R2")
-			(pintype "passive+no_connect")
+			(pintype "passive")
 		)
 		(pad "4" thru_hole circle
@@
 			(layers "*.Cu" "*.Mask")
 			(remove_unused_layers no)
-			(net 37 "unconnected-(RN1-R3-Pad4)")
+			(net 15 "Net-(A1-A1)")
 			(pinfunction "R3")
-			(pintype "passive+no_connect")
+			(pintype "passive")
 		)
 		(pad "5" thru_hole circle
@@
 			(layers "*.Cu" "*.Mask")
 			(remove_unused_layers no)
-			(net 18 "Net-(A1-A0)")
+			(net 11 "/m1_Vbat")
 			(pinfunction "R4")
 			(pintype "passive")
@@
 			(layers "*.Cu" "*.Mask")
 			(remove_unused_layers no)
-			(net 15 "Net-(A1-A1)")
+			(net 7 "/m2_Vbat")
 			(pinfunction "R5")
 			(pintype "passive")
@@
 			(layers "*.Cu" "*.Mask")
 			(remove_unused_layers no)
-			(net 11 "/m1_Vbat")
+			(net 14 "/m3_Vbat")
 			(pinfunction "R6")
 			(pintype "passive")
@@
 			(layers "*.Cu" "*.Mask")
 			(remove_unused_layers no)
-			(net 7 "/m2_Vbat")
-			(pinfunction "R7")
-			(pintype "passive")
-		)
-		(pad "9" thru_hole circle
-			(at 20.32 0 180)
-			(size 1.6 1.6)
-			(drill 0.8)
-			(layers "*.Cu" "*.Mask")
-			(remove_unused_layers no)
-			(net 14 "/m3_Vbat")
-			(pinfunction "R8")
-			(pintype "passive")
-		)
-		(pad "10" thru_hole circle
-			(at 22.86 0 180)
-			(size 1.6 1.6)
-			(drill 0.8)
-			(layers "*.Cu" "*.Mask")
-			(remove_unused_layers no)
 			(net 31 "/PUSH")
-			(pinfunction "R9")
+			(pinfunction "R7")
 			(pintype "passive")
 		)
 		(embedded_fonts no)
-		(model "${KICAD9_3DMODEL_DIR}/Resistor_THT.3dshapes/R_Array_SIP10.step"
+		(model "${KICAD9_3DMODEL_DIR}/Resistor_THT.3dshapes/R_Array_SIP8.step"
 			(offset
 				(xyz 0 0 0)
@@
 		(polygon
 			(pts
-				(xy 46.6815 28.906) (xy 46.6715 31.726) (xy 45.7715 31.726) (xy 45.5615 31.516) (xy 45.5615 30.646)
+				(xy 44.24 29.1) (xy 44.23 31.92) (xy 43.33 31.92) (xy 43.12 31.71) (xy 43.12 30.84)
 			)
 		)
