File: Kicad/SensorBoard/SensorBoard.kicad_sch (KiCad schematic)
At the start: 6 parts, among them J1 Conn_01x04, J2 Conn_01x02, U1 HCS-LSP-10A, U2 HCS-LSP-10A

Commit message: Update .cproject, .project, UPSMonitor.ino, and 29 more files
Connections:
- net +5V: now also J1.2 (Pin_2); no longer J1.1 (Pin_1)
- net Ibat: now also J1.4 (Pin_4); no longer J1.3 (Pin_3)
- net Iout: now also J1.3 (Pin_3); no longer J1.2 (Pin_2)
- net Vbat: now also J1.1 (Pin_1); no longer J1.4 (Pin_4)
Other:
- moved on the sheet: J1
Changed lines of the file:
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@@
 	(text "Monitoring Board"
 		(exclude_from_sim no)
-		(at 235.458 93.726 0)
+		(at 235.458 96.266 0)
 		(effects
 			(font
@@
 	)
 	(junction
-		(at 199.39 95.25)
+		(at 199.39 90.17)
 		(diameter 0)
 		(color 0 0 0 0)
@@
 	(wire
 		(pts
-			(xy 218.44 90.17) (xy 205.74 90.17)
-		)
-		(stroke
-			(width 0)
-			(type default)
-		)
-	)
-	(wire
-		(pts
-			(xy 217.17 87.63) (xy 218.44 87.63)
-		)
-		(stroke
-			(width 0)
-			(type default)
-		)
-	)
-	(wire
-		(pts
-			(xy 199.39 95.25) (xy 218.44 95.25)
+			(xy 213.36 97.79) (xy 218.44 97.79)
+		)
+		(stroke
+			(width 0)
+			(type default)
+		)
+	)
+	(wire
+		(pts
+			(xy 213.36 97.79) (xy 213.36 102.87)
+		)
+		(stroke
+			(width 0)
+			(type default)
+		)
+	)
+	(wire
+		(pts
+			(xy 212.09 86.36) (xy 212.09 92.71)
 		)
 		(stroke
@@
 	(wire
 		(pts
-			(xy 205.74 90.17) (xy 205.74 100.33)
-		)
-		(stroke
-			(width 0)
-			(type default)
-		)
-	)
-	(wire
-		(pts
 			(xy 144.78 85.09) (xy 144.78 86.36)
 		)
@@
 	(wire
 		(pts
-			(xy 199.39 95.25) (xy 199.39 97.79)
-		)
-		(stroke
-			(width 0)
-			(type default)
-		)
-	)
-	(wire
-		(pts
-			(xy 218.44 92.71) (xy 213.36 92.71)
-		)
-		(stroke
-			(width 0)
-			(type default)
-		)
-	)
-	(wire
-		(pts
 			(xy 218.44 74.93) (xy 218.44 76.2)
 		)
@@
 	(wire
 		(pts
+			(xy 212.09 92.71) (xy 218.44 92.71)
+		)
+		(stroke
+			(width 0)
+			(type default)
+		)
+	)
+	(wire
+		(pts
 			(xy 199.39 97.79) (xy 194.31 97.79)
 		)
@@
 	(wire
 		(pts
-			(xy 199.39 90.17) (xy 199.39 95.25)
+			(xy 199.39 90.17) (xy 199.39 97.79)
+		)
+		(stroke
+			(width 0)
+			(type default)
+		)
+	)
+	(wire
+		(pts
+			(xy 199.39 90.17) (xy 218.44 90.17)
+		)
+		(stroke
+			(width 0)
+			(type default)
+		)
+	)
+	(wire
+		(pts
+			(xy 205.74 95.25) (xy 218.44 95.25)
 		)
 		(stroke
@@
 	(wire
 		(pts
+			(xy 205.74 95.25) (xy 205.74 100.33)
+		)
+		(stroke
+			(width 0)
+			(type default)
+		)
+	)
+	(wire
+		(pts
 			(xy 153.67 96.52) (xy 153.67 102.87)
 		)
@@
 		)
 	)
-	(wire
-		(pts
-			(xy 213.36 92.71) (xy 213.36 102.87)
-		)
-		(stroke
-			(width 0)
-			(type default)
-		)
-	)
 	(label "Vbat"
+		(at 218.44 90.17 180)
+		(effects
+			(font
+				(size 1.27 1.27)
+			)
+			(justify right bottom)
+		)
+	)
+	(label "Ibat"
+		(at 218.44 97.79 180)
+		(effects
+			(font
+				(size 1.27 1.27)
+			)
+			(justify right bottom)
+		)
+	)
+	(label "Iout"
 		(at 218.44 95.25 180)
 		(effects
@@
 		)
 	)
-	(label "Ibat"
-		(at 218.44 92.71 180)
-		(effects
-			(font
-				(size 1.27 1.27)
-			)
-			(justify right bottom)
-		)
-	)
-	(label "Iout"
-		(at 218.44 90.17 180)
-		(effects
-			(font
-				(size 1.27 1.27)
-			)
-			(justify right bottom)
-		)
-	)
 	(symbol
 		(lib_id "power:+5V")
-		(at 217.17 87.63 0)
+		(at 212.09 86.36 0)
 		(unit 1)
 		(exclude_from_sim no)
@@
 		(dnp no)
 		(property "Reference" "#PWR01"
-			(at 217.17 91.44 0)
+			(at 212.09 90.17 0)
 			(effects
 				(font
@@
 		)
 		(property "Value" "+5V"
-			(at 214.376 85.598 0)
+			(at 209.296 84.328 0)
 			(effects
 				(font
@@
 		)
 		(property "Footprint" ""
-			(at 217.17 87.63 0)
+			(at 212.09 86.36 0)
 			(effects
 				(font
@@
 		)
 		(property "Datasheet" ""
-			(at 217.17 87.63 0)
+			(at 212.09 86.36 0)
 			(effects
 				(font
@@
 		)
 		(property "Description" "Power symbol creates a global label with name \"+5V\""
-			(at 217.17 87.63 0)
+			(at 212.09 86.36 0)
 			(effects
 				(font
@@
 	(symbol
 		(lib_id "Connector_Generic:Conn_01x04")
-		(at 223.52 90.17 0)
+		(at 223.52 92.71 0)
 		(unit 1)
 		(exclude_from_sim no)
@@
 		(fields_autoplaced yes)
 		(property "Reference" "J1"
-			(at 226.06 90.1699 0)
+			(at 226.06 92.7099 0)
 			(effects
 				(font
@@
 		)
 		(property "Value" "Conn_01x04"
-			(at 226.06 92.7099 0)
+			(at 226.06 95.2499 0)
 			(effects
 				(font
@@
 		)
 		(property "Footprint" "Connector_JST:JST_XH_B4B-XH-A_1x04_P2.50mm_Vertical"
-			(at 223.52 90.17 0)
+			(at 223.52 92.71 0)
 			(effects
 				(font
@@
 		)
 		(property "Datasheet" "~"
-			(at 223.52 90.17 0)
+			(at 223.52 92.71 0)
 			(effects
 				(font
@@
 		)
 		(property "Description" "Generic connector, single row, 01x04, script generated (kicad-library-utils/schlib/autogen/connector/)"
-			(at 223.52 90.17 0)
-			(effects
-				(font
+			(at 223.52 92.71 0)
+			(effects
+				(font
