File: Kicad/SensorBoard/SensorBoard.kicad_pcb (KiCad board)
At the start: 2 copper layers, 60.4 x 17.4 mm, 7 parts, among them J1 Conn_01x04, J2 Conn_01x02, U1 HCS-LSP-10A, U2 HCS-LSP-10A

Commit message: Update .cproject, .project, UPSMonitor.ino, and 29 more files
Connections:
- J1 pad 1: +5V -> /Vbat
- J1 pad 2: /Iout -> +5V
- J1 pad 3: /Ibat -> /Iout
- J1 pad 4: /Vbat -> /Ibat
- U1 pad : GND -> (no net)
Routing:
- net /Vbat: track 51.5 -> 37.0 mm
- net /Iout: track 7.07 -> 6.03 mm
- net /Ibat: track 41.6 -> 40.6 mm
Changed lines of the file:
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@@
 		(tags "Curren hall sensor open loop")
 		(property "Reference" "U1"
-			(at -5 0 0)
+			(at -2.815 5.525 0)
 			(layer "F.SilkS")
 			(effects
@@
 			)
 		)
-		(pad "" thru_hole roundrect
+		(pad "" np_thru_hole roundrect
 			(at 2.5 -0.55 180)
 			(size 3 3)
 			(drill 1)
 			(layers "*.Cu" "*.Mask")
-			(remove_unused_layers no)
 			(roundrect_rratio 0.1315789474)
-			(net 2 "GND")
-		)
-		(pad "" thru_hole roundrect
+		)
+		(pad "" np_thru_hole roundrect
 			(at 2.5 12.15 180)
 			(size 3 3)
 			(drill 1)
 			(layers "*.Cu" "*.Mask")
-			(remove_unused_layers no)
 			(roundrect_rratio 0.1388888889)
-			(net 2 "GND")
 		)
 		(pad "1" thru_hole oval
@@
 			(remove_unused_layers no)
 			(roundrect_rratio 0.147059)
-			(net 1 "+5V")
+			(net 4 "/Vbat")
 			(pinfunction "Pin_1")
 			(pintype "passive")
@@
 			(layers "*.Cu" "*.Mask")
 			(remove_unused_layers no)
-			(net 6 "/Iout")
+			(net 1 "+5V")
 			(pinfunction "Pin_2")
 			(pintype "passive")
@@
 			(layers "*.Cu" "*.Mask")
 			(remove_unused_layers no)
-			(net 5 "/Ibat")
+			(net 6 "/Iout")
 			(pinfunction "Pin_3")
 			(pintype "passive")
@@
 			(layers "*.Cu" "*.Mask")
 			(remove_unused_layers no)
-			(net 4 "/Vbat")
+			(net 5 "/Ibat")
 			(pinfunction "Pin_4")
 			(pintype "passive")
@@
 		(tags "Curren hall sensor open loop")
 		(property "Reference" "U2"
-			(at -5 0 0)
+			(at -0.77 5.055 0)
 			(layer "F.SilkS")
 			(effects
@@
 			)
 		)
-		(pad "" thru_hole roundrect
+		(pad "" np_thru_hole roundrect
 			(at 2.5 -0.55 180)
 			(size 3 3)
 			(drill 1)
 			(layers "*.Cu" "*.Mask")
-			(remove_unused_layers no)
 			(roundrect_rratio 0.1315789474)
 		)
-		(pad "" thru_hole roundrect
+		(pad "" np_thru_hole roundrect
 			(at 2.5 12.15 180)
 			(size 3 3)
 			(drill 1)
 			(layers "*.Cu" "*.Mask")
-			(remove_unused_layers no)
 			(roundrect_rratio 0.1388888889)
 		)
@@
 	)
 	(segment
+		(start 68.994039 52.280961)
+		(end 72.29 52.280961)
+		(width 1)
+		(layer "B.Cu")
+		(net 1)
+	)
+	(segment
+		(start 67.705 53.57)
+		(end 68.994039 52.280961)
+		(width 1)
+		(layer "B.Cu")
+		(net 1)
+	)
+	(segment
 		(start 45.027266 55.37)
 		(end 47.297266 53.1)
@@
 	)
 	(segment
-		(start 68.000961 54.780961)
-		(end 72.29 54.780961)
-		(width 1)
-		(layer "B.Cu")
-		(net 1)
-	)
-	(segment
 		(start 36.92 53.59)
 		(end 37.461961 54.131961)
@@
 	)
 	(segment
-		(start 66.79 53.57)
-		(end 68.000961 54.780961)
-		(width 1)
-		(layer "B.Cu")
-		(net 1)
-	)
-	(segment
 		(start 36.92 53.59)
 		(end 37.09 53.59)
@@
 	)
 	(segment
+		(start 66.79 53.57)
+		(end 67.705 53.57)
+		(width 1)
+		(layer "B.Cu")
+		(net 1)
+	)
+	(segment
 		(start 22.81 47.91)
 		(end 22.81 44.39)
@@
 	)
 	(segment
-		(start 72.96 57.87)
-		(end 75.08 55.75)
-		(width 1)
-		(layer "B.Cu")
-		(net 4)
-	)
-	(segment
 		(start 61.07096 54.753695)
-		(end 64.187265 57.87)
+		(end 62.558633 56.241367)
 		(width 1)
 		(layer "B.Cu")
@@
 	)
 	(segment
-		(start 74.265 47.280961)
-		(end 72.29 47.280961)
-		(width 1)
-		(layer "B.Cu")
-		(net 4)
-	)
-	(segment
-		(start 64.187265 57.87)
-		(end 72.96 57.87)
-		(width 1)
-		(layer "B.Cu")
-		(net 4)
-	)
-	(segment
 		(start 44.75 57.77)
 		(end 47.766305 54.753695)
@@
 	)
 	(segment
-		(start 75.08 48.095961)
-		(end 74.265 47.280961)
+		(start 62.558633 56.241367)
+		(end 70.829594 56.241367)
 		(width 1)
 		(layer "B.Cu")
@@
 	)
 	(segment
-		(start 75.08 55.75)
-		(end 75.08 48.095961)
+		(start 70.829594 56.241367)
+		(end 72.29 54.780961)
 		(width 1)
 		(layer "B.Cu")
 		(net 4)
+	)
+	(segment
+		(start 71.239 46.589)
+		(end 71.930961 47.280961)
+		(width 1)
+		(layer "B.Cu")
+		(net 5)
 	)
 	(segment
@@
 	)
 	(segment
-		(start 71.219653 49.780961)
-		(end 72.29 49.780961)
-		(width 1)
-		(layer "B.Cu")
-		(net 5)
-	)
-	(segment
-		(start 68.027692 46.589)
-		(end 71.219653 49.780961)
-		(width 1)
-		(layer "B.Cu")
-		(net 5)
-	)
-	(segment
-		(start 68.027692 46.589)
-		(end 61.642552 46.589)
-		(width 1)
-		(layer "B.Cu")
-		(net 5)
-	)
-	(segment
 		(start 36.92 48.51)
 		(end 37.311 48.119)
@@
 	)
 	(segment
+		(start 61.642552 46.589)
+		(end 71.239 46.589)
+		(width 1)
+		(layer "B.Cu")
+		(net 5)
+	)
+	(segment
+		(start 71.930961 47.280961)
+		(end 72.29 47.280961)
+		(width 1)
+		(layer "B.Cu")
+		(net 5)
+	)
+	(segment
 		(start 37.311 48.119)
 		(end 60.112552 48.119)
@@
 	)
 	(segment
-		(start 67.805958 48.49)
-		(end 71.596919 52.280961)
+		(start 70.030961 49.780961)
+		(end 68.74 48.49)
 		(width 1)
 		(layer "B.Cu")
@@
 	)
 	(segment
-		(start 66.79 48.49)
-		(end 67.805958 48.49)
+		(start 72.29 49.780961)
+		(end 70.030961 49.780961)
 		(width 1)
 		(layer "B.Cu")
@@
 	)
 	(segment
-		(start 71.596919 52.280961)
-		(end 72.29 52.280961)
-		(width 1)
-		(layer "B.Cu")
+		(start 68.74 48.49)
+		(end 66.79 48.49)
+		(width 1)
+		(layer "B.Cu")

Commit message: Update .sproject, io.cpp, io.h, and 29 more files
Other:
- board text added: "IK5PWC"
Changed lines of the file:
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@@
 			)
 		)
-		(pad "" np_thru_hole roundrect
+		(pad "" thru_hole roundrect
 			(at 2.5 -0.55 180)
 			(size 3 3)
 			(drill 1)
 			(layers "*.Cu" "*.Mask")
+			(remove_unused_layers no)
 			(roundrect_rratio 0.1315789474)
 		)
-		(pad "" np_thru_hole roundrect
+		(pad "" thru_hole roundrect
 			(at 2.5 12.15 180)
 			(size 3 3)
 			(drill 1)
 			(layers "*.Cu" "*.Mask")
+			(remove_unused_layers no)
 			(roundrect_rratio 0.1388888889)
 		)
@@
 			)
 		)
-		(pad "" np_thru_hole roundrect
+		(pad "" thru_hole roundrect
 			(at 2.5 -0.55 180)
 			(size 3 3)
 			(drill 1)
 			(layers "*.Cu" "*.Mask")
+			(remove_unused_layers no)
 			(roundrect_rratio 0.1315789474)
 		)
-		(pad "" np_thru_hole roundrect
+		(pad "" thru_hole roundrect
 			(at 2.5 12.15 180)
 			(size 3 3)
 			(drill 1)
 			(layers "*.Cu" "*.Mask")
+			(remove_unused_layers no)
 			(roundrect_rratio 0.1388888889)
 		)
@@
 		(layer "Edge.Cuts")
 	)
+	(gr_text "IK5PWC"
+		(at 20.525 43.15 90)
+		(layer "B.Cu")
+		(effects
+			(font
+				(size 2.8 2.8)
+				(thickness 0.7)
+				(bold yes)
+			)
+			(justify left bottom mirror)
+		)
+	)
 	(segment
 		(start 38.87 55.37)
@@
 			)
 		)
+	)
+	(zone
+		(net 0)
+		(net_name "")
+		(layer "B.Cu")
+		(hatch edge 0.5)
+		(connect_pads
+			(clearance 0)
+		)
+		(min_thickness 0.25)
+		(filled_areas_thickness no)
+		(keepout
+			(tracks not_allowed)
+			(vias not_allowed)
+			(pads not_allowed)
+			(copperpour not_allowed)
+			(footprints allowed)
+		)
+		(placement
+			(enabled no)
+			(sheetname "")
+		)
+		(fill
+			(thermal_gap 0.5)
+			(thermal_bridge_width 0.5)
+		)
+		(polygon
+			(pts
+				(xy 37.25 55.2) (xy 37.25 56.75) (xy 39.25 56.75) (xy 39.4 56.6) (xy 38 55.2)
+			)
+		)
